Commit message: chrore: improve the launch configuration

File: description/camera.xacro (robot description, xacro)
@@ -48,7 +48,4 @@
             <topic>camera/image_raw</topic>
             <gz_frame_id>camera_link_optical</gz_frame_id>
-            <!-- <plugin name="camera_controller" filename="libgazebo_ros_camera.so">
-                <frame_name>camera_link_optical</frame_name>
-            </plugin> -->
         </sensor>
     </gazebo>

File: description/gazebo_control.xacro (robot description, xacro)
@@ -7,5 +7,4 @@
             <wheel_separation>0.297</wheel_separation>
             <wheel_radius>0.033</wheel_radius>
-            <!-- <odom_publish_frequency>1</odom_publish_frequency> -->
             <topic>cmd_vel</topic>
             <max_linear_acceleration>0.33</max_linear_acceleration>
@@ -17,24 +16,4 @@
              <tf_topic>/tf</tf_topic>
         </plugin>
-        <!-- <plugin filename="gz-sim-joint-state-publisher-system"
-            name="gz::sim::systems::JointStatePublisher">
-            <topic>joint_states</topic>
-            <joint_name>left_wheel_joint</joint_name>
-            <joint_name>right_wheel_joint</joint_name>
-        </plugin> -->
     </gazebo>
-    <!-- <gazebo reference="chassis">
-       <material>Gazebo/Orange</material>
-    </gazebo>
-    <gazebo reference="caster_wheel">
-       <material>Gazebo/Black</material>
-       <mu1 value="0.001"/>
-       <mu2 value="0.001"/>
-    </gazebo>
-    <gazebo reference="right_wheel">
-        <material>Gazebo/Blue</material>
-    </gazebo>
-    <gazebo reference="left_wheel">
-        <material>Gazebo/Blue</material>
-    </gazebo> -->
 </robot>
